File: bms/bms.kicad_sch (KiCad schematic)
At the start: 39 parts, among them J10 Conn_02x10_Odd_Even, J11 Conn_02x08_Odd_Even, J12 Conn_02x10_Odd_Even, J13 Conn_02x08_Odd_Even, J14 Conn_02x08_Odd_Even, J15 Conn_02x10_Odd_Even, J3 Conn_01x10_Socket, J4 Conn_01x08_Socket, J5 Conn_01x08_Socket, J6 Conn_01x06_Socket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

Commit message: Revision / date added
Other:
- title: (none) -> Shield VCU - BMS
Changed lines of the file:
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@@
 	(generator_version "10.0")
 	(paper "A4")
+	(title_block
+		(title "Shield VCU - BMS")
+		(date "2026-05-26")
+		(rev "Viorel Stoica")
+	)
 	(rectangle
 		(start 203.2 30.48)

Commit message: CAN_IN & CAN_OUT - added
Parts:
- removed H1, H2, H3, H4: MountingHole_Pad, MountingHole:MountingHole_3.2mm_M3_ISO14580_Pad, symbol Mechanical:MountingHole_Pad
- added CAN_IN1: Conn_01x02_Pin, Connector_JST:JST_PH_B2B-PH-K_1x02_P2.00mm_Vertical, symbol Connector:Conn_01x02_Pin
- added D14: LED, LED_SMD:LED_0805_2012Metric, symbol Device:LED
- added R54: 1k, Resistor_SMD:R_1206_3216Metric_Pad1.30x1.75mm_HandSolder, symbol Device:R_Small
- B1: value Conn_01x02_Pin -> Supply
- CAN_OUT1: renamed from CAN_Bus_VCU1; footprint Connector_JST:JST_PH_S2B-PH-K_1x02_P2.00mm_Horizontal -> Connector_JST:JST_PH_B2B-PH-K_1x02_P2.00mm_Vertical
Connections:
- net 5V is gone; now on net 5V1: 5Vdd1.1 (Pin_1), 5Vdd1.2 (Pin_2), J3.6 (Pin_6)
- net 5V1: now also R54.1
- net CAN_H_k: now also CAN_IN1.1 (Pin_1)
- net CAN_L_k: now also CAN_IN1.2 (Pin_2)
- net GND: now also D14.1 (K)
- new net: D14.2 (A), R54.2
Other:
- note removed: "Mounting Holes"
- moved on the sheet: CAN_OUT1, CAN_k312
