File: bms/bms.kicad_sch (KiCad schematic)
At the start: 38 parts, among them J10 Conn_02x10_Odd_Even, J11 Conn_02x08_Odd_Even, J12 Conn_02x10_Odd_Even, J13 Conn_02x08_Odd_Even, J14 Conn_02x08_Odd_Even, J15 Conn_02x10_Odd_Even, J3 Conn_01x10_Socket, J4 Conn_01x08_Socket, J5 Conn_01x08_Socket, J6 Conn_01x06_Socket, U1 TLV76150DCY

Commit message: Traces correction+AMS Conn added
Parts:
- added CS1: CS, TestPoint:TestPoint_Loop_D2.50mm_Drill1.0mm, symbol Connector:TestPoint
- added Conn_AMS1: Conn_01x02_Pin, Connector_JST:JST_EH_B2B-EH-A_1x02_P2.50mm_Vertical, symbol Connector:Conn_01x02_Pin
- added GND1: GND, TestPoint:TestPoint_Loop_D2.50mm_Drill1.0mm, symbol Connector:TestPoint
- added MISO1: MISO, TestPoint:TestPoint_Loop_D2.50mm_Drill1.0mm, symbol Connector:TestPoint
- added SCK1: SCK, TestPoint:TestPoint_Loop_D2.50mm_Drill1.0mm, symbol Connector:TestPoint
- added SOUT1: SOUT, TestPoint:TestPoint_Loop_D2.50mm_Drill1.0mm, symbol Connector:TestPoint
- D1: value SS32 -> SK34; footprint Diode_THT:D_A-405_P7.62mm_Horizontal -> Diode_SMD:D_SMA_Handsoldering
Connections:
- net 1: now also Conn_Thermistors_1.8 (Pin_8), Conn_Thermistors_2.8 (Pin_8), Conn_Thermistors_3.8 (Pin_8), Conn_Thermistors_4.8 (Pin_8), Conn_Thermistors_5.8 (Pin_8), Conn_Thermistors_6.8 (Pin_8), Conn_Thermistors_7.8 (Pin_8), Conn_Thermistors_8.8 (Pin_8), J11.13 (Pin_13); no longer Conn_Thermistors_1.1 (Pin_1), Conn_Thermistors_2.1 (Pin_1), Conn_Thermistors_3.1 (Pin_1), Conn_Thermistors_4.1 (Pin_1), Conn_Thermistors_5.1 (Pin_1), Conn_Thermistors_6.1 (Pin_1), Conn_Thermistors_7.1 (Pin_1), Conn_Thermistors_8.1 (Pin_1), J14.1 (Pin_1)
- net 2: now also Conn_Thermistors_1.1 (Pin_1), Conn_Thermistors_2.1 (Pin_1), Conn_Thermistors_3.1 (Pin_1), Conn_Thermistors_4.1 (Pin_1), Conn_Thermistors_5.1 (Pin_1), Conn_Thermistors_6.1 (Pin_1), Conn_Thermistors_7.1 (Pin_1), Conn_Thermistors_8.1 (Pin_1); no longer Conn_Thermistors_1.2 (Pin_2), Conn_Thermistors_2.2 (Pin_2), Conn_Thermistors_3.2 (Pin_2), Conn_Thermistors_4.2 (Pin_2), Conn_Thermistors_5.2 (Pin_2), Conn_Thermistors_6.2 (Pin_2), Conn_Thermistors_7.2 (Pin_2), Conn_Thermistors_8.2 (Pin_2)
- net 3: now also Conn_Thermistors_1.2 (Pin_2), Conn_Thermistors_2.2 (Pin_2), Conn_Thermistors_3.2 (Pin_2), Conn_Thermistors_4.2 (Pin_2), Conn_Thermistors_5.2 (Pin_2), Conn_Thermistors_6.2 (Pin_2), Conn_Thermistors_7.2 (Pin_2), Conn_Thermistors_8.2 (Pin_2); no longer Conn_Thermistors_1.3 (Pin_3), Conn_Thermistors_2.3 (Pin_3), Conn_Thermistors_3.3 (Pin_3), Conn_Thermistors_4.3 (Pin_3), Conn_Thermistors_5.3 (Pin_3), Conn_Thermistors_6.3 (Pin_3), Conn_Thermistors_7.3 (Pin_3), Conn_Thermistors_8.3 (Pin_3)
- net 4: now also Conn_Thermistors_1.3 (Pin_3), Conn_Thermistors_2.3 (Pin_3), Conn_Thermistors_3.3 (Pin_3), Conn_Thermistors_4.3 (Pin_3), Conn_Thermistors_5.3 (Pin_3), Conn_Thermistors_6.3 (Pin_3), Conn_Thermistors_7.3 (Pin_3), Conn_Thermistors_8.3 (Pin_3); no longer Conn_Thermistors_1.4 (Pin_4), Conn_Thermistors_2.4 (Pin_4), Conn_Thermistors_3.4 (Pin_4), Conn_Thermistors_4.4 (Pin_4), Conn_Thermistors_5.4 (Pin_4), Conn_Thermistors_6.4 (Pin_4), Conn_Thermistors_7.4 (Pin_4), Conn_Thermistors_8.4 (Pin_4)
- net 5: now also Conn_Thermistors_1.4 (Pin_4), Conn_Thermistors_2.4 (Pin_4), Conn_Thermistors_3.4 (Pin_4), Conn_Thermistors_4.4 (Pin_4), Conn_Thermistors_5.4 (Pin_4), Conn_Thermistors_6.4 (Pin_4), Conn_Thermistors_7.4 (Pin_4), Conn_Thermistors_8.4 (Pin_4); no longer Conn_Thermistors_1.5 (Pin_5), Conn_Thermistors_2.5 (Pin_5), Conn_Thermistors_3.5 (Pin_5), Conn_Thermistors_4.5 (Pin_5), Conn_Thermistors_5.5 (Pin_5), Conn_Thermistors_6.5 (Pin_5), Conn_Thermistors_7.5 (Pin_5), Conn_Thermistors_8.5 (Pin_5)
- net 5V1: now also J4.2 (Pin_2); no longer J3.6 (Pin_6)
- net 6: now also Conn_Thermistors_1.5 (Pin_5), Conn_Thermistors_2.5 (Pin_5), Conn_Thermistors_3.5 (Pin_5), Conn_Thermistors_4.5 (Pin_5), Conn_Thermistors_5.5 (Pin_5), Conn_Thermistors_6.5 (Pin_5), Conn_Thermistors_7.5 (Pin_5), Conn_Thermistors_8.5 (Pin_5); no longer Conn_Thermistors_1.6 (Pin_6), Conn_Thermistors_2.6 (Pin_6), Conn_Thermistors_3.6 (Pin_6), Conn_Thermistors_4.6 (Pin_6), Conn_Thermistors_5.6 (Pin_6), Conn_Thermistors_6.6 (Pin_6), Conn_Thermistors_7.6 (Pin_6), Conn_Thermistors_8.6 (Pin_6)
- net 7: now also Conn_Thermistors_1.6 (Pin_6), Conn_Thermistors_2.6 (Pin_6), Conn_Thermistors_3.6 (Pin_6), Conn_Thermistors_4.6 (Pin_6), Conn_Thermistors_5.6 (Pin_6), Conn_Thermistors_6.6 (Pin_6), Conn_Thermistors_7.6 (Pin_6), Conn_Thermistors_8.6 (Pin_6); no longer Conn_Thermistors_1.7 (Pin_7), Conn_Thermistors_2.7 (Pin_7), Conn_Thermistors_3.7 (Pin_7), Conn_Thermistors_4.7 (Pin_7), Conn_Thermistors_5.7 (Pin_7), Conn_Thermistors_6.7 (Pin_7), Conn_Thermistors_7.7 (Pin_7), Conn_Thermistors_8.7 (Pin_7)
- net 8: now also Conn_Thermistors_1.7 (Pin_7), Conn_Thermistors_2.7 (Pin_7), Conn_Thermistors_3.7 (Pin_7), Conn_Thermistors_4.7 (Pin_7), Conn_Thermistors_5.7 (Pin_7), Conn_Thermistors_6.7 (Pin_7), Conn_Thermistors_7.7 (Pin_7), Conn_Thermistors_8.7 (Pin_7); no longer Conn_Thermistors_1.8 (Pin_8), Conn_Thermistors_2.8 (Pin_8), Conn_Thermistors_3.8 (Pin_8), Conn_Thermistors_4.8 (Pin_8), Conn_Thermistors_5.8 (Pin_8), Conn_Thermistors_6.8 (Pin_8), Conn_Thermistors_7.8 (Pin_8), Conn_Thermistors_8.8 (Pin_8)
- net CS: now also J10.5 (Pin_5), J3.8 (Pin_8), CS1.1; no longer J10.11 (Pin_11), J3.2 (Pin_2)
- net G05: now also J12.1 (Pin_1); no longer J10.12 (Pin_12)
- net G06: now also J12.3 (Pin_3); no longer J10.10 (Pin_10)
- net G07: now also J11.8 (Pin_8); no longer J10.8 (Pin_8)
- net G08: now also J11.6 (Pin_6); no longer J10.6 (Pin_6)
- net GND: now also J3.4 (Pin_4), GND1.1; no longer J3.8 (Pin_8)
- net MISO: now also J10.9 (Pin_9), J3.6 (Pin_6), MISO1.1; no longer J10.7 (Pin_7), J3.4 (Pin_4)
- net SCK: now also J10.11 (Pin_11), SCK1.1; no longer J10.5 (Pin_5)
- net SOUT: now also J10.7 (Pin_7), J3.7 (Pin_7), SOUT1.1; no longer J10.9 (Pin_9), J3.3 (Pin_3)
- net Reserved: now reaches J15.18 (Pin_18)
- net Reserved: now also Conn_AMS1.1 (Pin_1)
- net AMS: now reaches J15.20 (Pin_20)
- net AMS: now also Conn_AMS1.2 (Pin_2)
- no-connect marks 106 -> 102
Other:
- moved on the sheet: CAN_IMD1
