File: bms/bms.kicad_pcb (KiCad board)
At the start: 2 copper layers, 87.2 x 156.6 mm, 37 parts, among them J10 Conn_02x10_Odd_Even, J11 Conn_02x08_Odd_Even, J12 Conn_02x10_Odd_Even, J13 Conn_02x08_Odd_Even, J14 Conn_02x08_Odd_Even, J15 Conn_02x10_Odd_Even, J3 Conn_01x10_Socket, J4 Conn_01x08_Socket, J5 Conn_01x08_Socket, J6 Conn_01x06_Socket, U1 TLV76150DCY

Commit message: Traces correction+AMS Conn added
Parts:
- added CS1: CS, TestPoint:TestPoint_Loop_D2.50mm_Drill1.0mm, F.Cu at (119.7, 115.7)
- added Conn_AMS1: Conn_01x02_Pin, Connector_JST:JST_EH_B2B-EH-A_1x02_P2.50mm_Vertical, F.Cu at (73.7, 177.3)
- added GND1: GND, TestPoint:TestPoint_Loop_D2.50mm_Drill1.0mm, F.Cu at (55.4, 37.2)
- added MISO1: MISO, TestPoint:TestPoint_Loop_D2.50mm_Drill1.0mm, F.Cu at (119.7, 106.7)
- added SCK1: SCK, TestPoint:TestPoint_Loop_D2.50mm_Drill1.0mm, F.Cu at (119.7, 102.8)
- added SOUT1: SOUT, TestPoint:TestPoint_Loop_D2.50mm_Drill1.0mm, F.Cu at (119.7, 111.4)
- D1: value SS32 -> SK34; footprint Diode_THT:D_A-405_P7.62mm_Horizontal -> Diode_SMD:D_SMA_Handsoldering
- moved Soft_G_B5-6 56.5 mm to (127.0, 165.9)
- moved Soft_G_B11-12 12.1 mm to (127.0, 137.6)
- moved Soft_G_B15-16 12.1 mm to (127.0, 155.6)
- moved Soft_G_B13-14 12.1 mm to (127.0, 146.6)
- moved Soft_G_B9-10 12.1 mm to (127.0, 128.7)
- moved D1 1.33 mm to (61.1, 49.7), turned to 90 degrees
- moved Soft_G_B7-8 1.01 mm to (126.9, 119.3)
Connections:
- Conn_Thermistors_1 pad 1: 1 -> 2
- Conn_Thermistors_1 pad 2: 2 -> 3
- Conn_Thermistors_1 pad 3: 3 -> 4
- Conn_Thermistors_1 pad 4: 4 -> 5
- Conn_Thermistors_1 pad 5: 5 -> 6
- Conn_Thermistors_1 pad 6: 6 -> 7
- Conn_Thermistors_1 pad 7: 7 -> 8
- Conn_Thermistors_1 pad 8: 8 -> 1
- Conn_Thermistors_2 pad 1: 1 -> 2
- Conn_Thermistors_2 pad 2: 2 -> 3
- Conn_Thermistors_2 pad 3: 3 -> 4
- Conn_Thermistors_2 pad 4: 4 -> 5
- Conn_Thermistors_2 pad 5: 5 -> 6
- Conn_Thermistors_2 pad 6: 6 -> 7
- Conn_Thermistors_2 pad 7: 7 -> 8
- Conn_Thermistors_2 pad 8: 8 -> 1
- Conn_Thermistors_3 pad 1: 1 -> 2
- Conn_Thermistors_3 pad 2: 2 -> 3
- Conn_Thermistors_3 pad 3: 3 -> 4
- Conn_Thermistors_3 pad 4: 4 -> 5
- Conn_Thermistors_3 pad 5: 5 -> 6
- Conn_Thermistors_3 pad 6: 6 -> 7
- Conn_Thermistors_3 pad 7: 7 -> 8
- Conn_Thermistors_3 pad 8: 8 -> 1
- Conn_Thermistors_4 pad 1: 1 -> 2
- Conn_Thermistors_4 pad 2: 2 -> 3
- Conn_Thermistors_4 pad 3: 3 -> 4
- Conn_Thermistors_4 pad 4: 4 -> 5
- Conn_Thermistors_4 pad 5: 5 -> 6
- Conn_Thermistors_4 pad 6: 6 -> 7
- Conn_Thermistors_4 pad 7: 7 -> 8
- Conn_Thermistors_4 pad 8: 8 -> 1
- Conn_Thermistors_5 pad 1: 1 -> 2
- Conn_Thermistors_5 pad 2: 2 -> 3
- Conn_Thermistors_5 pad 3: 3 -> 4
- Conn_Thermistors_5 pad 4: 4 -> 5
- Conn_Thermistors_5 pad 5: 5 -> 6
- Conn_Thermistors_5 pad 6: 6 -> 7
- Conn_Thermistors_5 pad 7: 7 -> 8
- Conn_Thermistors_5 pad 8: 8 -> 1
- Conn_Thermistors_6 pad 1: 1 -> 2
- Conn_Thermistors_6 pad 2: 2 -> 3
- Conn_Thermistors_6 pad 3: 3 -> 4
- Conn_Thermistors_6 pad 4: 4 -> 5
- Conn_Thermistors_6 pad 5: 5 -> 6
- Conn_Thermistors_6 pad 6: 6 -> 7
- Conn_Thermistors_6 pad 7: 7 -> 8
- Conn_Thermistors_6 pad 8: 8 -> 1
- Conn_Thermistors_7 pad 1: 1 -> 2
- Conn_Thermistors_7 pad 2: 2 -> 3
- Conn_Thermistors_7 pad 3: 3 -> 4
- Conn_Thermistors_7 pad 4: 4 -> 5
- Conn_Thermistors_7 pad 5: 5 -> 6
- Conn_Thermistors_7 pad 6: 6 -> 7
- Conn_Thermistors_7 pad 7: 7 -> 8
- Conn_Thermistors_7 pad 8: 8 -> 1
- Conn_Thermistors_8 pad 1: 1 -> 2
- Conn_Thermistors_8 pad 2: 2 -> 3
- Conn_Thermistors_8 pad 3: 3 -> 4
- Conn_Thermistors_8 pad 4: 4 -> 5
- Conn_Thermistors_8 pad 5: 5 -> 6
- Conn_Thermistors_8 pad 6: 6 -> 7
- Conn_Thermistors_8 pad 7: 7 -> 8
- Conn_Thermistors_8 pad 8: 8 -> 1
- J10 pad 10: G06 -> unconnected-(J10-Pin_10-Pad10)
- J10 pad 11: CS -> SCK
- J10 pad 12: G05 -> unconnected-(J10-Pin_12-Pad12)
- J10 pad 5: SCK -> CS
- J10 pad 6: G08 -> unconnected-(J10-Pin_6-Pad6)
- J10 pad 7: MISO -> SOUT
- J10 pad 8: G07 -> unconnected-(J10-Pin_8-Pad8)
- J10 pad 9: SOUT -> MISO
- J11 pad 13: unconnected-(J11-Pin_13-Pad13) -> 1
- J11 pad 6: unconnected-(J11-Pin_6-Pad6) -> G08
- J11 pad 8: unconnected-(J11-Pin_8-Pad8) -> G07
- J12 pad 1: unconnected-(J12-Pin_1-Pad1) -> G05
- J12 pad 3: unconnected-(J12-Pin_3-Pad3) -> G06
- J14 pad 1: 1 -> unconnected-(J14-Pin_1-Pad1)
- J15 pad 18: unconnected-(J15-Pin_18-Pad18) -> Reserved
- J15 pad 20: unconnected-(J15-Pin_20-Pad20) -> AMS
- J3 pad 2: CS -> unconnected-(J3-Pin_2-Pad2)
- J3 pad 3: SOUT -> unconnected-(J3-Pin_3-Pad3)
- J3 pad 4: MISO -> GND
- J3 pad 6: 5V1 -> MISO
- J3 pad 7: unconnected-(J3-Pin_7-Pad7) -> SOUT
- J3 pad 8: GND -> CS
- J4 pad 2: unconnected-(J4-Pin_2-Pad2) -> 5V1
Routing:
- net 5V1: track 155.9 -> 49.7 mm
- net GND: track 33.8 -> 14.0 mm, vias 5 -> 3
- net Reserved: track 0.00 -> 17.7 mm
- net CS: track 9.09 -> 23.2 mm
- net AMS: track 0.00 -> 13.3 mm
- net SOUT: track 9.09 -> 21.7 mm
- net MISO: track 9.09 -> 20.0 mm
- net SCK: track 9.63 -> 19.4 mm
- net 4: track 114.0 -> 121.5 mm
- net G06: track 14.4 -> 21.9 mm
- net G10: track 12.5 -> 19.0 mm
- net G09: track 12.5 -> 18.8 mm
- net G14: track 12.1 -> 16.3 mm
- net G13: track 12.1 -> 16.3 mm
- net 1: track 103.2 -> 107.4 mm
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Other:
- board text added: "AMS_OUT"
- board text added: "BAT+"
- board text added: "GND"
- board text added: "SUPPLY"
- board text added: "VCU_BMS V1.1"
- board text removed: "VCU_BMS V1.0"
